File: grape/io.sch (KiCad schematic (older format))
At the start: 59 parts

Commit message: Annotation added
Parts:
- gave numbers to parts that had none: 55

Commit message: Footprint assignment and some additions
Parts:
- C15, C16, C17, C18, C19, C20, C21, C22, C23, C24, C25, C26, C27, C28, C29, C30, C31, C32, C33, C34, C35, C36: footprint (none) -> Capacitor_SMD:C_0805_2012Metric_Pad1.18x1.45mm_HandSolder
- J3, J4, J5, J6, J7: footprint (none) -> Connector_Audio:Jack_3.5mm_QingPu_WQP-PJ398SM_Vertical_CircularHoles
- R10, R11, R12, R13, R14, R15, R16, R17, R18, R19, R20, R4, R5, R6, R7, R8, R9: footprint (none) -> Resistor_SMD:R_0805_2012Metric_Pad1.20x1.40mm_HandSolder
- RV1, RV2, RV3, RV4, RV5: footprint (none) -> Potentiometer_THT:Potentiometer_Alps_RK09L_Single_Vertical
- TP2, TP3, TP4: footprint (none) -> TestPoint:TestPoint_Pad_D1.5mm
- U3: footprint PW20 -> Package_SO:TSSOP-20_4.4x6.5mm_P0.65mm
- U4: footprint (none) -> Package_SO:TSSOP-14_4.4x5mm_P0.65mm
- U5: footprint (none) -> Package_SO:SO-8_5.3x6.2mm_P1.27mm
