File: grape/power.sch (KiCad schematic (older format))
At the start: 22 parts

Commit message: Annotation added
Parts:
- gave numbers to parts that had none: 22
Changed lines of the file:
@@
 $EndDescr
 $Comp
-L Connector_Generic:Conn_02x05_Counter_Clockwise J?
+L Connector_Generic:Conn_02x05_Counter_Clockwise J8
 U 1 1 5FC78DA2
 P 3450 3850
-F 0 "J?" H 3500 4267 50  0000 C CNN
+F 0 "J8" H 3500 4267 50  0000 C CNN
 F 1 "Conn_02x05_Counter_Clockwise" H 3500 4176 50  0000 C CNN
 F 2 "" H 3450 3850 50  0001 C CNN
@@
 $EndComp
 $Comp
-L power:GND #PWR?
+L power:GND #PWR078
 U 1 1 5FC7997B
 P 3250 4050
-F 0 "#PWR?" H 3250 3800 50  0001 C CNN
+F 0 "#PWR078" H 3250 3800 50  0001 C CNN
 F 1 "GND" H 3255 3877 50  0000 C CNN
 F 2 "" H 3250 4050 50  0001 C CNN
@@
 $EndComp
 $Comp
-L power:GND #PWR?
+L power:GND #PWR077
 U 1 1 5FC7A86D
 P 3250 3850
-F 0 "#PWR?" H 3250 3600 50  0001 C CNN
+F 0 "#PWR077" H 3250 3600 50  0001 C CNN
 F 1 "GND" V 3255 3722 50  0000 R CNN
 F 2 "" H 3250 3850 50  0001 C CNN
@@
 $EndComp
 $Comp
-L power:GND #PWR?
+L power:GND #PWR079
 U 1 1 5FC7AD8F
 P 3750 3950
-F 0 "#PWR?" H 3750 3700 50  0001 C CNN
+F 0 "#PWR079" H 3750 3700 50  0001 C CNN
 F 1 "GND" V 3755 3822 50  0000 R CNN
 F 2 "" H 3750 3950 50  0001 C CNN
@@
 NoConn ~ 3750 4050
 $Comp
-L Device:D D?
+L Device:D D34
 U 1 1 5FC7B66D
 P 3900 3650
-F 0 "D?" H 3900 3433 50  0000 C CNN
+F 0 "D34" H 3900 3433 50  0000 C CNN
 F 1 "D" H 3900 3524 50  0000 C CNN
 F 2 "" H 3900 3650 50  0001 C CNN
@@
 $EndComp
 $Comp
-L Device:D D?
+L Device:D D35
 U 1 1 5FC7C64A
 P 3900 4500
-F 0 "D?" H 3900 4717 50  0000 C CNN
+F 0 "D35" H 3900 4717 50  0000 C CNN
 F 1 "D" H 3900 4626 50  0000 C CNN
 F 2 "" H 3900 4500 50  0001 C CNN
@@
 	2850 4500 3750 4500
 $Comp
-L Device:C_Polarized C?
+L Device:C_Polarized C37
 U 1 1 5FC7EB05
 P 4700 3800
-F 0 "C?" H 4818 3846 50  0000 L CNN
+F 0 "C37" H 4818 3846 50  0000 L CNN
 F 1 "50u" H 4818 3755 50  0000 L CNN
 F 2 "" H 4738 3650 50  0001 C CNN
@@
 $EndComp
 $Comp
-L Device:C_Polarized C?
+L Device:C_Polarized C38
 U 1 1 5FC7F16D
 P 4700 4250
-F 0 "C?" H 4582 4204 50  0000 R CNN
+F 0 "C38" H 4582 4204 50  0000 R CNN
 F 1 "50u" H 4582 4295 50  0000 R CNN
 F 2 "" H 4738 4100 50  0001 C CNN
@@
 $EndComp
 $Comp
-L power:VCC #PWR?
+L power:VCC #PWR080
 U 1 1 5FC7FCC4
 P 4700 3500
-F 0 "#PWR?" H 4700 3350 50  0001 C CNN
+F 0 "#PWR080" H 4700 3350 50  0001 C CNN
 F 1 "VCC" H 4715 3673 50  0000 C CNN
 F 2 "" H 4700 3500 50  0001 C CNN
@@
 $EndComp
 $Comp
-L power:VEE #PWR?
+L power:VEE #PWR082
 U 1 1 5FC7FFFB
 P 4700 4600
-F 0 "#PWR?" H 4700 4450 50  0001 C CNN
+F 0 "#PWR082" H 4700 4450 50  0001 C CNN
 F 1 "VEE" H 4715 4773 50  0000 C CNN
 F 2 "" H 4700 4600 50  0001 C CNN
@@
 $EndComp
 $Comp
-L Device:R R?
+L Device:R R21
 U 1 1 5FC810DD
 P 5450 4500
-F 0 "R?" V 5243 4500 50  0000 C CNN
+F 0 "R21" V 5243 4500 50  0000 C CNN
 F 1 "2.2k" V 5334 4500 50  0000 C CNN
 F 2 "" V 5380 4500 50  0001 C CNN
@@
 $EndComp
 $Comp
-L Reference_Voltage:LM4040DBZ-10 U?
+L Reference_Voltage:LM4040DBZ-10 U6
 U 1 1 5FC82BFD
 P 5800 4700
-F 0 "U?" V 5750 4400 50  0000 L CNN
+F 0 "U6" V 5750 4400 50  0000 L CNN
 F 1 "LM4040DBZ-10" V 5850 4050 50  0000 L CNN
 F 2 "Package_TO_SOT_SMD:SOT-23" H 5800 4500 50  0001 C CIN
@@
 $EndComp
 $Comp
-L Device:C C?
+L Device:C C39
 U 1 1 5FC84064
 P 6300 4700
-F 0 "C?" H 6415 4746 50  0000 L CNN
+F 0 "C39" H 6415 4746 50  0000 L CNN
 F 1 "10u" H 6415 4655 50  0000 L CNN
 F 2 "" H 6338 4550 50  0001 C CNN
@@
 $EndComp
 $Comp
-L Device:C C?
+L Device:C C41
 U 1 1 5FC84898
 P 6800 4700
-F 0 "C?" H 6915 4746 50  0000 L CNN
+F 0 "C41" H 6915 4746 50  0000 L CNN
 F 1 "100n" H 6915 4655 50  0000 L CNN
 F 2 "" H 6838 4550 50  0001 C CNN
@@
 	6300 4950 6800 4950
 $Comp
-L power:GND #PWR?
+L power:GND #PWR083
 U 1 1 5FC87381
 P 5950 4950
-F 0 "#PWR?" H 5950 4700 50  0001 C CNN
+F 0 "#PWR083" H 5950 4700 50  0001 C CNN
 F 1 "GND" H 5955 4777 50  0000 C CNN
 F 2 "" H 5950 4950 50  0001 C CNN
@@
 	4700 3950 4700 4050
 $Comp
-L power:GND #PWR?
+L power:GND #PWR081
 U 1 1 5FC87F3F
 P 4700 4050
-F 0 "#PWR?" H 4700 3800 50  0001 C CNN
+F 0 "#PWR081" H 4700 3800 50  0001 C CNN
 F 1 "GND" V 4705 3922 50  0000 R CNN
 F 2 "" H 4700 4050 50  0001 C CNN
@@
 	4700 4050 4700 4100
 $Comp
-L Regulator_Switching:R-78E3.3-0.5 U?
+L Regulator_Switching:R-78E3.3-0.5 U7
 U 1 1 5FC88A85
 P 7550 2200
-F 0 "U?" H 7550 2442 50  0000 C CNN
+F 0 "U7" H 7550 2442 50  0000 C CNN
 F 1 "R-78E3.3-0.5" H 7550 2351 50  0000 C CNN
 F 2 "Converter_DCDC:Converter_DCDC_RECOM_R-78E-0.5_THT" H 7600 1950 50  0001 L CIN
@@
 $EndComp
 $Comp
-L Device:L L?
+L Device:L L4
 U 1 1 5FC8C889
 P 6850 2200
-F 0 "L?" V 7040 2200 50  0000 C CNN
+F 0 "L4" V 7040 2200 50  0000 C CNN
 F 1 "33uH" V 6949 2200 50  0000 C CNN
 F 2 "" H 6850 2200 50  0001 C CNN
@@
 $EndComp
 $Comp
-L Device:C C?
+L Device:C C42
 U 1 1 5FC8D048
 P 7100 2350
-F 0 "C?" H 7215 2396 50  0000 L CNN
+F 0 "C42" H 7215 2396 50  0000 L CNN
 F 1 "22u" H 7215 2305 50  0000 L CNN
 F 2 "" H 7138 2200 50  0001 C CNN
@@
 $EndComp
 $Comp
-L Device:C C?
+L Device:C C40
 U 1 1 5FC8DB36
 P 6500 2350
-F 0 "C?" H 6615 2396 50  0000 L CNN
+F 0 "C40" H 6615 2396 50  0000 L CNN
 F 1 "22u" H 6615 2305 50  0000 L CNN
 F 2 "" H 6538 2200 50  0001 C CNN
@@
 $EndComp
 $Comp
-L Device:C C?
+L Device:C C44
 U 1 1 5FC8DFB5
 P 8150 2350
-F 0 "C?" H 8265 2396 50  0000 L CNN
+F 0 "C44" H 8265 2396 50  0000 L CNN
 F 1 "100n" H 8265 2305 50  0000 L CNN
 F 2 "" H 8188 2200 50  0001 C CNN
@@
 $EndComp
 $Comp
-L Device:C_Polarized C?
+L Device:C_Polarized C45
 U 1 1 5FC8E743
 P 8600 2350
-F 0 "C?" H 8718 2396 50  0000 L CNN
+F 0 "C45" H 8718 2396 50  0000 L CNN
 F 1 "50u" H 8718 2305 50  0000 L CNN
 F 2 "" H 8638 2200 50  0001 C CNN
@@
 Connection ~ 8150 2200
 $Comp
-L power:GND #PWR?
+L power:GND #PWR084
 U 1 1 5FC8FD3C
 P 6500 2500
-F 0 "#PWR?" H 6500 2250 50  0001 C CNN
+F 0 "#PWR084" H 6500 2250 50  0001 C CNN
 F 1 "GND" H 6505 2327 50  0000 C CNN
 F 2 "" H 6500 2500 50  0001 C CNN
@@
 $EndComp
 $Comp
-L power:GND #PWR?
+L power:GND #PWR085
 U 1 1 5FC900E4
 P 7100 2500
-F 0 "#PWR?" H 7100 2250 50  0001 C CNN
+F 0 "#PWR085" H 7100 2250 50  0001 C CNN
 F 1 "GND" H 7105 2327 50  0000 C CNN
 F 2 "" H 7100 2500 50  0001 C CNN
@@
 $EndComp
 $Comp
-L power:GND #PWR?
+L power:GND #PWR086
 U 1 1 5FC903E4
 P 7550 2500
-F 0 "#PWR?" H 7550 2250 50  0001 C CNN
+F 0 "#PWR086" H 7550 2250 50  0001 C CNN
 F 1 "GND" H 7555 2327 50  0000 C CNN
 F 2 "" H 7550 2500 50  0001 C CNN
@@
 $EndComp
 $Comp
-L power:GND #PWR?
+L power:GND #PWR089
 U 1 1 5FC90B04
 P 8150 2500
-F 0 "#PWR?" H 8150 2250 50  0001 C CNN
+F 0 "#PWR089" H 8150 2250 50  0001 C CNN
 F 1 "GND" H 8155 2327 50  0000 C CNN
 F 2 "" H 8150 2500 50  0001 C CNN
@@
 $EndComp
 $Comp
-L power:GND #PWR?
+L power:GND #PWR091
 U 1 1 5FC90CE5
 P 8600 2500
-F 0 "#PWR?" H 8600 2250 50  0001 C CNN
+F 0 "#PWR091" H 8600 2250 50  0001 C CNN
 F 1 "GND" H 8605 2327 50  0000 C CNN
 F 2 "" H 8600 2500 50  0001 C CNN
@@
 $EndComp
 $Comp
-L power:+3.3V #PWR?
+L power:+3.3V #PWR090
 U 1 1 5FC9112C
 P 8350 2200
-F 0 "#PWR?" H 8350 2050 50  0001 C CNN
+F 0 "#PWR090" H 8350 2050 50  0001 C CNN
 F 1 "+3.3V" H 8365 2373 50  0000 C CNN
 F 2 "" H 8350 2200 50  0001 C CNN
@@
 Connection ~ 6800 4500
 $Comp
-L Device:L L?
+L Device:L L3
 U 1 1 5FC9381D
 P 6800 3300
-F 0 "L?" V 6990 3300 50  0000 C CNN
+F 0 "L3" V 6990 3300 50  0000 C CNN
 F 1 "L" V 6899 3300 50  0000 C CNN
 F 2 "" H 6800 3300 50  0001 C CNN
@@
 $EndComp
 $Comp
-L Regulator_Linear:MIC5205-3.3YM5 U?
+L Regulator_Linear:MIC5205-3.3YM5 U8
 U 1 1 5FC95B35
 P 7550 3400
-F 0 "U?" H 7550 3742 50  0000 C CNN
+F 0 "U8" H 7550 3742 50  0000 C CNN
 F 1 "MIC5205-3.3YM5" H 7550 3651 50  0000 C CNN
 F 2 "Package_TO_SOT_SMD:SOT-23-5" H 7550 3725 50  0001 C CNN
@@
 $EndComp
 $Comp
-L Device:C C?
+L Device:C C43
 U 1 1 5FC986C8
 P 8050 3550
-F 0 "C?" H 8165 3596 50  0000 L CNN
+F 0 "C43" H 8165 3596 50  0000 L CNN
 F 1 "470pF" H 8165 3505 50  0000 L CNN
 F 2 "" H 8088 3400 50  0001 C CNN
@@
 	7100 3300 7250 3300
 $Comp
-L power:GND #PWR?
+L power:GND #PWR087
 U 1 1 5FC99AB1
 P 7550 3700
-F 0 "#PWR?" H 7550 3450 50  0001 C CNN
+F 0 "#PWR087" H 7550 3450 50  0001 C CNN
 F 1 "GND" H 7555 3527 50  0000 C CNN
 F 2 "" H 7550 3700 50  0001 C CNN
@@
 $EndComp
 $Comp
-L power:GND #PWR?
+L power:GND #PWR088
 U 1 1 5FC99F93
 P 8050 3700
-F 0 "#PWR?" H 8050 3450 50  0001 C CNN
+F 0 "#PWR088" H 8050 3450 50  0001 C CNN
 F 1 "GND" H 8055 3527 50  0000 C CNN
 F 2 "" H 8050 3700 50  0001 C CNN
@@
 	5800 2200 6500 2200
 $Comp
-L Device:L L?
+L Device:L L1
 U 1 1 5FC9CA67
 P 4350 3650
-F 0 "L?" V 4540 3650 50  0000 C CNN
+F 0 "L1" V 4540 3650 50  0000 C CNN
 F 1 "L" V 4449 3650 50  0000 C CNN
 F 2 "" H 4350 3650 50  0001 C CNN
@@
 $EndComp
 $Comp
-L Device:L L?
+L Device:L L2
 U 1 1 5FC9E2F5
 P 4350 4500
-F 0 "L?" V 4540 4500 50  0000 C CNN
+F 0 "L2" V 4540 4500 50  0000 C CNN
 F 1 "L" V 4449 4500 50  0000 C CNN
 F 2 "" H 4350 4500 50  0001 C CNN
@@
 $EndComp
 $Comp
-L power:+3.3VA #PWR?
+L power:+3.3VA #PWR093
 U 1 1 5FC9EA25
 P 8800 3300
-F 0 "#PWR?" H 8800 3150 50  0001 C CNN
+F 0 "#PWR093" H 8800 3150 50  0001 C CNN
 F 1 "+3.3VA" H 8815 3473 50  0000 C CNN
 F 2 "" H 8800 3300 50  0001 C CNN
@@
 $EndComp
 $Comp
-L Device:C C?
+L Device:C C46
 U 1 1 5FE350AC
 P 8600 3550
-F 0 "C?" H 8715 3596 50  0000 L CNN
+F 0 "C46" H 8715 3596 50  0000 L CNN
 F 1 "100n" H 8715 3505 50  0000 L CNN
 F 2 "" H 8638 3400 50  0001 C CNN
@@
 $EndComp
 $Comp
-L Device:C_Polarized C?
+L Device:C_Polarized C47
 U 1 1 5FE350B2
 P 9050 3550
-F 0 "C?" H 9168 3596 50  0000 L CNN
+F 0 "C47" H 9168 3596 50  0000 L CNN
 F 1 "50u" H 9168 3505 50  0000 L CNN
 F 2 "" H 9088 3400 50  0001 C CNN
@@
 $EndComp
 $Comp
-L power:GND #PWR?
+L power:GND #PWR092
 U 1 1 5FE350B8
 P 8600 3700
-F 0 "#PWR?" H 8600 3450 50  0001 C CNN
+F 0 "#PWR092" H 8600 3450 50  0001 C CNN
 F 1 "GND" H 8605 3527 50  0000 C CNN
 F 2 "" H 8600 3700 50  0001 C CNN
@@
 $EndComp
 $Comp
-L power:GND #PWR?
+L power:GND #PWR094
 U 1 1 5FE350BE
 P 9050 3700
-F 0 "#PWR?" H 9050 3450 50  0001 C CNN
+F 0 "#PWR094" H 9050 3450 50  0001 C CNN
 F 1 "GND" H 9055 3527 50  0000 C CNN
 F 2 "" H 9050 3700 50  0001 C CNN

Commit message: Footprint assignment and some additions
Parts:
- C37, C38, C45, C46: footprint (none) -> Capacitor_Tantalum_SMD:CP_EIA-7343-31_Kemet-D_Pad2.25x2.55mm_HandSolder
- C39, C40, C41, C42, C43, C44: footprint (none) -> Capacitor_SMD:C_0805_2012Metric_Pad1.18x1.45mm_HandSolder
- C47: footprint (none) -> Capacitor_Tantalum_SMD:CP_EIA-7343-30_AVX-N_Pad2.25x2.55mm_HandSolder
- D34, D35: footprint (none) -> Diode_SMD:D_SMA-SMB_Universal_Handsoldering
- J8: footprint (none) -> Connector_IDC:IDC-Header_2x05_P2.54mm_Vertical
- L1, L2, L3: footprint (none) -> Capacitor_SMD:C_1206_3216Metric_Pad1.33x1.80mm_HandSolder
- L4: footprint (none) -> Inductor_SMD:L_Sumida_CDMC6D28_7.25x6.5mm
- R21: footprint (none) -> Resistor_SMD:R_0805_2012Metric_Pad1.20x1.40mm_HandSolder
Changed lines of the file:
@@
 F 0 "J8" H 3500 4267 50  0000 C CNN
 F 1 "Conn_02x05_Counter_Clockwise" H 3500 4176 50  0000 C CNN
-F 2 "" H 3450 3850 50  0001 C CNN
+F 2 "Connector_IDC:IDC-Header_2x05_P2.54mm_Vertical" H 3450 3850 50  0001 C CNN
 F 3 "~" H 3450 3850 50  0001 C CNN
 	1    3450 3850
@@
 F 0 "D34" H 3900 3433 50  0000 C CNN
 F 1 "D" H 3900 3524 50  0000 C CNN
-F 2 "" H 3900 3650 50  0001 C CNN
+F 2 "Diode_SMD:D_SMA-SMB_Universal_Handsoldering" H 3900 3650 50  0001 C CNN
 F 3 "~" H 3900 3650 50  0001 C CNN
 	1    3900 3650
@@
 F 0 "D35" H 3900 4717 50  0000 C CNN
 F 1 "D" H 3900 4626 50  0000 C CNN
-F 2 "" H 3900 4500 50  0001 C CNN
+F 2 "Diode_SMD:D_SMA-SMB_Universal_Handsoldering" H 3900 4500 50  0001 C CNN
 F 3 "~" H 3900 4500 50  0001 C CNN
 	1    3900 4500
@@
 F 0 "C37" H 4818 3846 50  0000 L CNN
 F 1 "50u" H 4818 3755 50  0000 L CNN
-F 2 "" H 4738 3650 50  0001 C CNN
+F 2 "Capacitor_Tantalum_SMD:CP_EIA-7343-31_Kemet-D_Pad2.25x2.55mm_HandSolder" H 4738 3650 50  0001 C CNN
 F 3 "~" H 4700 3800 50  0001 C CNN
 	1    4700 3800
@@
 F 0 "C38" H 4582 4204 50  0000 R CNN
 F 1 "50u" H 4582 4295 50  0000 R CNN
-F 2 "" H 4738 4100 50  0001 C CNN
+F 2 "Capacitor_Tantalum_SMD:CP_EIA-7343-31_Kemet-D_Pad2.25x2.55mm_HandSolder" H 4738 4100 50  0001 C CNN
 F 3 "~" H 4700 4250 50  0001 C CNN
 	1    4700 4250
@@
 F 0 "R21" V 5243 4500 50  0000 C CNN
 F 1 "2.2k" V 5334 4500 50  0000 C CNN
-F 2 "" V 5380 4500 50  0001 C CNN
+F 2 "Resistor_SMD:R_0805_2012Metric_Pad1.20x1.40mm_HandSolder" V 5380 4500 50  0001 C CNN
 F 3 "~" H 5450 4500 50  0001 C CNN
 	1    5450 4500
@@
 F 0 "C39" H 6415 4746 50  0000 L CNN
 F 1 "10u" H 6415 4655 50  0000 L CNN
-F 2 "" H 6338 4550 50  0001 C CNN
+F 2 "Capacitor_SMD:C_0805_2012Metric_Pad1.18x1.45mm_HandSolder" H 6338 4550 50  0001 C CNN
 F 3 "~" H 6300 4700 50  0001 C CNN
 	1    6300 4700
@@
 F 0 "C41" H 6915 4746 50  0000 L CNN
 F 1 "100n" H 6915 4655 50  0000 L CNN
-F 2 "" H 6838 4550 50  0001 C CNN
+F 2 "Capacitor_SMD:C_0805_2012Metric_Pad1.18x1.45mm_HandSolder" H 6838 4550 50  0001 C CNN
 F 3 "~" H 6800 4700 50  0001 C CNN
 	1    6800 4700
@@
 F 0 "L4" V 7040 2200 50  0000 C CNN
 F 1 "33uH" V 6949 2200 50  0000 C CNN
-F 2 "" H 6850 2200 50  0001 C CNN
+F 2 "Inductor_SMD:L_Sumida_CDMC6D28_7.25x6.5mm" H 6850 2200 50  0001 C CNN
 F 3 "~" H 6850 2200 50  0001 C CNN
 	1    6850 2200
@@
 F 0 "C42" H 7215 2396 50  0000 L CNN
 F 1 "22u" H 7215 2305 50  0000 L CNN
-F 2 "" H 7138 2200 50  0001 C CNN
+F 2 "Capacitor_SMD:C_0805_2012Metric_Pad1.18x1.45mm_HandSolder" H 7138 2200 50  0001 C CNN
 F 3 "~" H 7100 2350 50  0001 C CNN
 	1    7100 2350
@@
 F 0 "C40" H 6615 2396 50  0000 L CNN
 F 1 "22u" H 6615 2305 50  0000 L CNN
-F 2 "" H 6538 2200 50  0001 C CNN
+F 2 "Capacitor_SMD:C_0805_2012Metric_Pad1.18x1.45mm_HandSolder" H 6538 2200 50  0001 C CNN
 F 3 "~" H 6500 2350 50  0001 C CNN
 	1    6500 2350
@@
 F 0 "C44" H 8265 2396 50  0000 L CNN
 F 1 "100n" H 8265 2305 50  0000 L CNN
-F 2 "" H 8188 2200 50  0001 C CNN
+F 2 "Capacitor_SMD:C_0805_2012Metric_Pad1.18x1.45mm_HandSolder" H 8188 2200 50  0001 C CNN
 F 3 "~" H 8150 2350 50  0001 C CNN
 	1    8150 2350
@@
 F 0 "C45" H 8718 2396 50  0000 L CNN
 F 1 "50u" H 8718 2305 50  0000 L CNN
-F 2 "" H 8638 2200 50  0001 C CNN
+F 2 "Capacitor_Tantalum_SMD:CP_EIA-7343-31_Kemet-D_Pad2.25x2.55mm_HandSolder" H 8638 2200 50  0001 C CNN
 F 3 "~" H 8600 2350 50  0001 C CNN
 	1    8600 2350
@@
 F 0 "L3" V 6990 3300 50  0000 C CNN
 F 1 "L" V 6899 3300 50  0000 C CNN
-F 2 "" H 6800 3300 50  0001 C CNN
+F 2 "Capacitor_SMD:C_1206_3216Metric_Pad1.33x1.80mm_HandSolder" H 6800 3300 50  0001 C CNN
 F 3 "~" H 6800 3300 50  0001 C CNN
 	1    6800 3300
@@
 F 0 "C43" H 8165 3596 50  0000 L CNN
 F 1 "470pF" H 8165 3505 50  0000 L CNN
-F 2 "" H 8088 3400 50  0001 C CNN
+F 2 "Capacitor_SMD:C_0805_2012Metric_Pad1.18x1.45mm_HandSolder" H 8088 3400 50  0001 C CNN
 F 3 "~" H 8050 3550 50  0001 C CNN
 	1    8050 3550
@@
 F 0 "L1" V 4540 3650 50  0000 C CNN
 F 1 "L" V 4449 3650 50  0000 C CNN
-F 2 "" H 4350 3650 50  0001 C CNN
+F 2 "Capacitor_SMD:C_1206_3216Metric_Pad1.33x1.80mm_HandSolder" H 4350 3650 50  0001 C CNN
 F 3 "~" H 4350 3650 50  0001 C CNN
 	1    4350 3650
@@
 F 0 "L2" V 4540 4500 50  0000 C CNN
 F 1 "L" V 4449 4500 50  0000 C CNN
-F 2 "" H 4350 4500 50  0001 C CNN
+F 2 "Capacitor_SMD:C_1206_3216Metric_Pad1.33x1.80mm_HandSolder" H 4350 4500 50  0001 C CNN
 F 3 "~" H 4350 4500 50  0001 C CNN
 	1    4350 4500
@@
 F 0 "C46" H 8715 3596 50  0000 L CNN
 F 1 "100n" H 8715 3505 50  0000 L CNN
-F 2 "" H 8638 3400 50  0001 C CNN
+F 2 "Capacitor_Tantalum_SMD:CP_EIA-7343-31_Kemet-D_Pad2.25x2.55mm_HandSolder" H 8638 3400 50  0001 C CNN
 F 3 "~" H 8600 3550 50  0001 C CNN
 	1    8600 3550
@@
 F 0 "C47" H 9168 3596 50  0000 L CNN
 F 1 "50u" H 9168 3505 50  0000 L CNN
-F 2 "" H 9088 3400 50  0001 C CNN
+F 2 "Capacitor_Tantalum_SMD:CP_EIA-7343-30_AVX-N_Pad2.25x2.55mm_HandSolder" H 9088 3400 50  0001 C CNN
 F 3 "~" H 9050 3550 50  0001 C CNN
 	1    9050 3550
