File: grape/core.sch (KiCad schematic (older format))
At the start: 59 parts

Commit message: Annotation added
Parts:
- gave numbers to parts that had none: 59

Commit message: Footprint assignment and some additions
Parts:
- added H1, H2, H3, H4: MountingHole, MountingHole:MountingHole_3.2mm_M3_Pad_Via, symbol Mechanical:MountingHole
- C1, C10, C11, C12, C13, C14, C2, C3, C4, C5, C6, C7, C8, C9: footprint (none) -> Capacitor_SMD:C_0805_2012Metric_Pad1.18x1.45mm_HandSolder
- D1, D10, D11, D12, D13, D14, D15, D16, D17, D18, D19, D2, D20, D21, D22, D23, D24, D25, D26, D27, D28, D29, D3, D30, D31, D32, D33, D4, D5, D6, D7, D8, D9: footprint (none) -> LED_THT:LED_D3.0mm
- J1: footprint (none) -> Connector_Molex:Molex_PicoBlade_53047-0310_1x03_P1.25mm_Vertical
- J2: footprint (none) -> Connector_Molex:Molex_PicoBlade_53047-0610_1x06_P1.25mm_Vertical
- R1, R2, R3: footprint (none) -> Resistor_SMD:R_0805_2012Metric_Pad1.20x1.40mm_HandSolder
- SW1, SW2, SW3: footprint (none) -> Button_Switch_SMD:SW_SPST_TL3305A
- TP1: footprint (none) -> TestPoint:TestPoint_Pad_D1.5mm
- Y1: value Crystal -> ABM3-8.000MHZ-D2Y-T; footprint (none) -> Crystal:Crystal_SMD_5032-2Pin_5.0x3.2mm_HandSoldering

Commit message: Routing in progress
Parts:
- removed D33: LED, LED_THT:LED_D3.0mm, symbol Device:LED
Connections:
- no-connect marks 15 -> 16
Changed lines of the file:
@@
-	1    0    0    -1
-$EndComp
-$Comp
-L Device:LED D33
-U 1 1 5FCD28F6
-P 10700 5100
-F 0 "D33" H 10693 5317 50  0000 C CNN
-F 1 "LED" H 10693 5226 50  0000 C CNN
-F 2 "LED_THT:LED_D3.0mm" H 10700 5100 50  0001 C CNN
-F 3 "~" H 10700 5100 50  0001 C CNN
-	1    10700 5100
 	1    0    0    -1
 $EndComp
@@
 Wire Wire Line
 	9500 5000 10150 5000
-Wire Wire Line
-	9500 5100 10550 5100
-Wire Wire Line
-	10850 5100 10850 5000
 Wire Wire Line
 	10850 1900 10000 1900
@@
 Wire Wire Line
 	10450 5000 10850 5000
-Connection ~ 10850 5000
 Wire Wire Line
 	10850 5000 10850 4900
@@
 	1    0    0    -1
 $EndComp
+NoConn ~ 9500 5100
 $EndSCHEMATC

Commit message: Finished routing
Connections:
- net at U1.2 (PC13): now also SW3.2
- net at U1.20 (PB2): no longer SW3.2
Changed lines of the file:
@@
 $EndComp
-Wire Wire Line
-	3750 3900 4550 3900
 Wire Wire Line
 	3250 4000 4550 4000
@@
 NoConn ~ 4550 4900
 NoConn ~ 4550 5000
-NoConn ~ 4550 3300
 NoConn ~ 4550 3400
 NoConn ~ 4550 3500
@@
 $EndComp
 NoConn ~ 9500 5100
+Wire Wire Line
+	3750 3900 4050 3900
+Wire Wire Line
+	4050 3900 4050 3300
+Wire Wire Line
+	4050 3300 4550 3300
+NoConn ~ 4550 3900
 $EndSCHEMATC
