File: grape/grape.kicad_pcb (KiCad board)
At the start: 2 copper layers, 70 x 110 mm, 0 parts

Commit message: Components placed
Parts:
- added C1: 100n, Capacitor_SMD:C_0805_2012Metric_Pad1.18x1.45mm_HandSolder, F.Cu at (156.5, 108.2)
- added C10: 100n, Capacitor_SMD:C_0805_2012Metric_Pad1.18x1.45mm_HandSolder, F.Cu at (160.5, 118.3)
- added C11: 1u, Capacitor_SMD:C_0805_2012Metric_Pad1.18x1.45mm_HandSolder, F.Cu at (176.8, 108.2)
- added C12: 1u, Capacitor_SMD:C_0805_2012Metric_Pad1.18x1.45mm_HandSolder, F.Cu at (162.6, 118.4)
- added C13: 1 uF, Capacitor_SMD:C_0805_2012Metric_Pad1.18x1.45mm_HandSolder, F.Cu at (160.0, 94.0)
- added C14: 1u, Capacitor_SMD:C_0805_2012Metric_Pad1.18x1.45mm_HandSolder, F.Cu at (164.5, 95.0)
- added C15: 100n, Capacitor_SMD:C_0805_2012Metric_Pad1.18x1.45mm_HandSolder, F.Cu at (127.0, 134.1)
- added C16: 10u, Capacitor_SMD:C_0805_2012Metric_Pad1.18x1.45mm_HandSolder, F.Cu at (140.2, 128.5)
- added C17: 100n, Capacitor_SMD:C_0805_2012Metric_Pad1.18x1.45mm_HandSolder, F.Cu at (129.0, 134.1)
- added C18: 100n, Capacitor_SMD:C_0805_2012Metric_Pad1.18x1.45mm_HandSolder, F.Cu at (140.2, 133.1)
- added C19: 10u, Capacitor_SMD:C_0805_2012Metric_Pad1.18x1.45mm_HandSolder, F.Cu at (128.5, 128.0)
- added C2: 100n, Capacitor_SMD:C_0805_2012Metric_Pad1.18x1.45mm_HandSolder, F.Cu at (156.5, 112.8)
- added C20: 100n, Capacitor_SMD:C_0805_2012Metric_Pad1.18x1.45mm_HandSolder, F.Cu at (143.3, 130.1)
- added C21: 1.0nF, Capacitor_SMD:C_0805_2012Metric_Pad1.18x1.45mm_HandSolder, F.Cu at (130.0, 151.0)
- added C22: 1.0nF, Capacitor_SMD:C_0805_2012Metric_Pad1.18x1.45mm_HandSolder, F.Cu at (155.0, 149.0)
- added C23: 1.0nF, Capacitor_SMD:C_0805_2012Metric_Pad1.18x1.45mm_HandSolder, F.Cu at (151.2, 132.5)
- added C24: 1.0nF, Capacitor_SMD:C_0805_2012Metric_Pad1.18x1.45mm_HandSolder, F.Cu at (163.2, 136.5)
- added C25: 2.2u, Capacitor_SMD:C_0805_2012Metric_Pad1.18x1.45mm_HandSolder, F.Cu at (128.0, 131.1)
- added C26: 2.2u, Capacitor_SMD:C_0805_2012Metric_Pad1.18x1.45mm_HandSolder, F.Cu at (134.6, 125.5)
- added C27: 1.0nF, Capacitor_SMD:C_0805_2012Metric_Pad1.18x1.45mm_HandSolder, F.Cu at (142.0, 148.0)
- added C28: 1.0nF, Capacitor_SMD:C_0805_2012Metric_Pad1.18x1.45mm_HandSolder, F.Cu at (166.5, 148.0)
- added C29: 1.0n, Capacitor_SMD:C_0805_2012Metric_Pad1.18x1.45mm_HandSolder, F.Cu at (119.4, 124.0)
- added C3: 100n, Capacitor_SMD:C_0805_2012Metric_Pad1.18x1.45mm_HandSolder, F.Cu at (162.6, 112.8)
- added C30: 1.0nF, Capacitor_SMD:C_0805_2012Metric_Pad1.18x1.45mm_HandSolder, F.Cu at (151.2, 137.5)
- added C31: 1.0nF, Capacitor_SMD:C_0805_2012Metric_Pad1.18x1.45mm_HandSolder, F.Cu at (163.2, 132.5)
- added C32: C, Capacitor_SMD:C_0805_2012Metric_Pad1.18x1.45mm_HandSolder, F.Cu at (112.8, 128.0)
- added C33: 100n, Capacitor_SMD:C_0805_2012Metric_Pad1.18x1.45mm_HandSolder, F.Cu at (151.4, 128.0)
- added C34: 100n, Capacitor_SMD:C_0805_2012Metric_Pad1.18x1.45mm_HandSolder, F.Cu at (117.4, 135.1)
- added C35: 10 u, Capacitor_SMD:C_0805_2012Metric_Pad1.18x1.45mm_HandSolder, F.Cu at (147.3, 128.0)
- added C36: 100n, Capacitor_SMD:C_0805_2012Metric_Pad1.18x1.45mm_HandSolder, F.Cu at (122.4, 135.1)
- added C37: 50u, Capacitor_Tantalum_SMD:CP_EIA-7343-31_Kemet-D_Pad2.25x2.55mm_HandSolder, F.Cu at (128.5, 117.0)
- added C38: 50u, Capacitor_Tantalum_SMD:CP_EIA-7343-31_Kemet-D_Pad2.25x2.55mm_HandSolder, F.Cu at (134.1, 117.0)
- added C39: 10u, Capacitor_SMD:C_0805_2012Metric_Pad1.18x1.45mm_HandSolder, F.Cu at (140.2, 123.4)
- added C4: 2.2uF, Capacitor_SMD:C_0805_2012Metric_Pad1.18x1.45mm_HandSolder, F.Cu at (170.8, 121.9)
- added C40: 22u, Capacitor_SMD:C_0805_2012Metric_Pad1.18x1.45mm_HandSolder, F.Cu at (134.1, 109.7)
- added C41: 100n, Capacitor_SMD:C_0805_2012Metric_Pad1.18x1.45mm_HandSolder, F.Cu at (143.3, 123.4)
- added C42: 22u, Capacitor_SMD:C_0805_2012Metric_Pad1.18x1.45mm_HandSolder, F.Cu at (127.5, 102.6)
- added C43: 470pF, Capacitor_SMD:C_0805_2012Metric_Pad1.18x1.45mm_HandSolder, F.Cu at (161.5, 128.0)
- added C44: 100n, Capacitor_SMD:C_0805_2012Metric_Pad1.18x1.45mm_HandSolder, F.Cu at (141.2, 103.6)
- added C45: 100n, Capacitor_SMD:C_0805_2012Metric_Pad1.18x1.45mm_HandSolder, F.Cu at (137.7, 108.7)
- added C46: 100n, Capacitor_SMD:C_0805_2012Metric_Pad1.18x1.45mm_HandSolder, F.Cu at (161.5, 126.0)
- added C47: 50u, Capacitor_Tantalum_SMD:CP_EIA-7343-30_AVX-N_Pad2.25x2.55mm_HandSolder, F.Cu at (175.3, 134.6)
- added C48: 50u, Capacitor_Tantalum_SMD:CP_EIA-7343-31_Kemet-D_Pad2.25x2.55mm_HandSolder, F.Cu at (149.4, 100.6)
- added C5: 100n, Capacitor_SMD:C_0805_2012Metric_Pad1.18x1.45mm_HandSolder, F.Cu at (178.8, 108.2)
- added C6: 1u, Capacitor_SMD:C_0805_2012Metric_Pad1.18x1.45mm_HandSolder, F.Cu at (174.9, 124.5)
- added C7: 100n, Capacitor_SMD:C_0805_2012Metric_Pad1.18x1.45mm_HandSolder, F.Cu at (174.9, 121.9)
- added C8: 1u, Capacitor_SMD:C_0805_2012Metric_Pad1.18x1.45mm_HandSolder, F.Cu at (168.1, 100.1)
- added C9: 100n, Capacitor_SMD:C_0805_2012Metric_Pad1.18x1.45mm_HandSolder, F.Cu at (168.1, 102.6)
- added D1: LED, LED_THT:LED_D3.0mm, F.Cu at (132.5, 60.0)
- added D10: LED, LED_THT:LED_D3.0mm, F.Cu at (132.5, 85.0)
- added D11: LED, LED_THT:LED_D3.0mm, F.Cu at (140.0, 80.0)
- added D12: LED, LED_THT:LED_D3.0mm, F.Cu at (155.0, 70.0)
- added D13: LED, LED_THT:LED_D3.0mm, F.Cu at (140.0, 90.0)
- added D14: LED, LED_THT:LED_D3.0mm, F.Cu at (155.0, 90.0)
- added D15: LED, LED_THT:LED_D3.0mm, F.Cu at (132.5, 70.0)
- added D16: LED, LED_THT:LED_D3.0mm, F.Cu at (155.0, 80.0)
- added D17: LED, LED_THT:LED_D3.0mm, F.Cu at (132.5, 80.0)
- added D18: LED, LED_THT:LED_D3.0mm, F.Cu at (140.0, 75.0)
- added D19: LED, LED_THT:LED_D3.0mm, F.Cu at (147.5, 70.0)
- added D2: LED, LED_THT:LED_D3.0mm, F.Cu at (147.5, 85.0)
- added D20: LED, LED_THT:LED_D3.0mm, F.Cu at (147.5, 90.0)
- added D21: LED, LED_THT:LED_D3.0mm, F.Cu at (132.5, 65.0)
- added D22: LED, LED_THT:LED_D3.0mm, F.Cu at (155.0, 85.0)
- added D23: LED, LED_THT:LED_D3.0mm, F.Cu at (132.5, 90.0)
- added D24: LED, LED_THT:LED_D3.0mm, F.Cu at (175.0, 87.5)
- added D25: LED, LED_THT:LED_D3.0mm, F.Cu at (140.0, 70.0)
- added D26: LED, LED_THT:LED_D3.0mm, F.Cu at (155.0, 55.0)
- added D27: LED, LED_THT:LED_D3.0mm, F.Cu at (140.0, 65.0)
- added D28: LED, LED_THT:LED_D3.0mm, F.Cu at (140.0, 60.0)
- added D29: LED, LED_THT:LED_D3.0mm, F.Cu at (140.0, 85.0)
- added D3: LED, LED_THT:LED_D3.0mm, F.Cu at (147.5, 65.0)
- added D30: LED, LED_THT:LED_D3.0mm, F.Cu at (147.5, 80.0)
- added D31: LED, LED_THT:LED_D3.0mm, F.Cu at (132.5, 55.0)
- added D32: LED, LED_THT:LED_D3.0mm, F.Cu at (140.0, 55.0)
- added D33: LED, LED_THT:LED_D3.0mm, F.Cu at (147.5, 75.0)
- added D34: D, Diode_SMD:D_SMA-SMB_Universal_Handsoldering, F.Cu at (122.5, 106.8)
- added D35: D, Diode_SMD:D_SMA-SMB_Universal_Handsoldering, F.Cu at (122.5, 117.0)
- added D4: LED, LED_THT:LED_D3.0mm, F.Cu at (132.5, 75.0)
- added D5: LED, LED_THT:LED_D3.0mm, F.Cu at (155.0, 75.0)
- added D6: LED, LED_THT:LED_D3.0mm, F.Cu at (155.0, 60.0)
- added D7: LED, LED_THT:LED_D3.0mm, F.Cu at (147.5, 60.0)
- added D8: LED, LED_THT:LED_D3.0mm, F.Cu at (147.5, 55.0)
- added D9: LED, LED_THT:LED_D3.0mm, F.Cu at (155.0, 65.0)
- added H1: MountingHole, MountingHole:MountingHole_3.2mm_M3_Pad_Via, F.Cu at (176.5, 48.5)
- added H2: MountingHole, MountingHole:MountingHole_3.2mm_M3_Pad_Via, F.Cu at (113.5, 48.5)
- added H3: MountingHole, MountingHole:MountingHole_3.2mm_M3_Pad_Via, F.Cu at (176.5, 151.5)
- added H4: MountingHole, MountingHole:MountingHole_3.2mm_M3_Pad_Via, F.Cu at (113.5, 151.5)
- added J1: UART, Connector_Molex:Molex_PicoBlade_53047-0310_1x03_P1.25mm_Vertical, F.Cu at (148.3, 121.4)
- added J2: SWD, Connector_Molex:Molex_PicoBlade_53047-0610_1x06_P1.25mm_Vertical, F.Cu at (144.8, 115.8)
- added J3: CV 1V/Oct, Connector_Audio:Jack_3.5mm_QingPu_WQP-PJ398SM_Vertical_CircularHoles, F.Cu at (134.0, 140.0)
- added J4: PARAM 1, Connector_Audio:Jack_3.5mm_QingPu_WQP-PJ398SM_Vertical_CircularHoles, F.Cu at (157.0, 140.0)
- added J5: WAVE CV, Connector_Audio:Jack_3.5mm_QingPu_WQP-PJ398SM_Vertical_CircularHoles, F.Cu at (145.5, 140.0)
- added J6: PARAM 2, Connector_Audio:Jack_3.5mm_QingPu_WQP-PJ398SM_Vertical_CircularHoles, F.Cu at (168.5, 140.0)
- added J7: AUDIO OUT, Connector_Audio:Jack_3.5mm_QingPu_WQP-PJ398SM_Vertical_CircularHoles, F.Cu at (121.5, 140.0)
- added J8: Conn_02x05_Counter_Clockwise, Connector_IDC:IDC-Header_2x05_P2.54mm_Vertical, F.Cu at (116.3, 116.3)
- added L1: L, Capacitor_SMD:C_1206_3216Metric_Pad1.33x1.80mm_HandSolder, F.Cu at (112.8, 138.2)
- added L2: L, Capacitor_SMD:C_1206_3216Metric_Pad1.33x1.80mm_HandSolder, F.Cu at (129.1, 123.4)
- added L3: L, Capacitor_SMD:C_1206_3216Metric_Pad1.33x1.80mm_HandSolder, F.Cu at (127.5, 108.2)
- added L4: 33uH, Inductor_SMD:L_Sumida_CDMC6D28_7.25x6.5mm, F.Cu at (134.1, 103.1)
- added L5: 33uH, Inductor_SMD:L_Sumida_CDMC6D28_7.25x6.5mm, F.Cu at (149.0, 107.2)
- added R1: R, Resistor_SMD:R_0805_2012Metric_Pad1.20x1.40mm_HandSolder, F.Cu at (157.5, 99.0)
- added R10: 1k, Resistor_SMD:R_0805_2012Metric_Pad1.20x1.40mm_HandSolder, F.Cu at (134.6, 135.6)
- added R11: 22k, Resistor_SMD:R_0805_2012Metric_Pad1.20x1.40mm_HandSolder, F.Cu at (123.4, 124.0)
- added R12: 100k, Resistor_SMD:R_0805_2012Metric_Pad1.20x1.40mm_HandSolder, F.Cu at (148.0, 148.0)
- added R13: 100k, Resistor_SMD:R_0805_2012Metric_Pad1.20x1.40mm_HandSolder, F.Cu at (173.5, 148.0)
- added R14: 100k, Resistor_SMD:R_0805_2012Metric_Pad1.20x1.40mm_HandSolder, F.Cu at (147.2, 137.5)
- added R15: 100k, Resistor_SMD:R_0805_2012Metric_Pad1.20x1.40mm_HandSolder, F.Cu at (167.2, 132.5)
- added R16: 10k, Resistor_SMD:R_0805_2012Metric_Pad1.20x1.40mm_HandSolder, F.Cu at (115.3, 124.0)
- added R17: 33k, Resistor_SMD:R_0805_2012Metric_Pad1.20x1.40mm_HandSolder, F.Cu at (149.2, 137.5)
- added R18: 33k, Resistor_SMD:R_0805_2012Metric_Pad1.20x1.40mm_HandSolder, F.Cu at (165.2, 132.5)
- added R19: 33k, Resistor_SMD:R_0805_2012Metric_Pad1.20x1.40mm_HandSolder, F.Cu at (112.8, 132.6)
- added R2: R, Resistor_SMD:R_0805_2012Metric_Pad1.20x1.40mm_HandSolder, F.Cu at (170.5, 95.0)
- added R20: 1k, Resistor_SMD:R_0805_2012Metric_Pad1.20x1.40mm_HandSolder, F.Cu at (123.0, 149.0)
- added R21: 2.2k, Resistor_SMD:R_0805_2012Metric_Pad1.20x1.40mm_HandSolder, F.Cu at (134.6, 122.9)
- added R22: R, Resistor_SMD:R_0805_2012Metric_Pad1.20x1.40mm_HandSolder, F.Cu at (141.2, 106.2)
- added R23: R, Resistor_SMD:R_0805_2012Metric_Pad1.20x1.40mm_HandSolder, F.Cu at (141.2, 108.2)
- added R3: R, Resistor_SMD:R_0805_2012Metric_Pad1.20x1.40mm_HandSolder, F.Cu at (157.5, 96.5)
- added R4: 100k, Resistor_SMD:R_0805_2012Metric_Pad1.20x1.40mm_HandSolder, F.Cu at (135.5, 150.0)
- added R5: 100k, Resistor_SMD:R_0805_2012Metric_Pad1.20x1.40mm_HandSolder, F.Cu at (161.0, 149.0)
- added R6: 100k, Resistor_SMD:R_0805_2012Metric_Pad1.20x1.40mm_HandSolder, F.Cu at (147.2, 132.5)
- added R7: 100k, Resistor_SMD:R_0805_2012Metric_Pad1.20x1.40mm_HandSolder, F.Cu at (167.2, 136.5)
- added R8: 33k, Resistor_SMD:R_0805_2012Metric_Pad1.20x1.40mm_HandSolder, F.Cu at (149.2, 132.5)
- added R9: 33k, Resistor_SMD:R_0805_2012Metric_Pad1.20x1.40mm_HandSolder, F.Cu at (165.2, 136.5)
- added RV1: PARAM_3, Potentiometer_THT:Potentiometer_Alps_RK09L_Single_Vertical, F.Cu at (165.0, 77.5)
- added RV2: PARAM_4, Potentiometer_THT:Potentiometer_Alps_RK09L_Single_Vertical, F.Cu at (115.0, 95.0)
- added RV3: FREQ, Potentiometer_THT:Potentiometer_Alps_RK09L_Single_Vertical, F.Cu at (115.0, 80.0)
- added RV4: WAVE_ONE, Potentiometer_THT:Potentiometer_Alps_RK09L_Single_Vertical, F.Cu at (115.0, 65.0)
- added RV5: WAVE_TWO, Potentiometer_THT:Potentiometer_Alps_RK09L_Single_Vertical, F.Cu at (165.0, 62.5)
- added SW1: PARAM_8, Button_Switch_SMD:SW_SPST_TL3305A, B.Cu at (165.0, 50.0)
- added SW2: PARAM_7, Button_Switch_SMD:SW_SPST_TL3305A, B.Cu at (122.5, 50.0)
- added SW3: PARAM_6, Button_Switch_SMD:SW_SPST_TL3305A, B.Cu at (145.0, 50.0)
- added TP1: TestPoint, TestPoint:TestPoint_Pad_D1.5mm, F.Cu at (173.2, 101.6)
- added TP2: TestPoint, TestPoint:TestPoint_Pad_D1.5mm, F.Cu at (165.6, 121.9)
- added TP3: TestPoint, TestPoint:TestPoint_Pad_D1.5mm, F.Cu at (177.8, 115.8)
- added TP4: TestPoint, TestPoint:TestPoint_Pad_D1.5mm, F.Cu at (177.8, 118.9)
- added U1: STM32F411CEUx, Package_DFN_QFN:QFN-48-1EP_7x7mm_P0.5mm_EP5.6x5.6mm, F.Cu at (170.2, 110.7)
- added U2: LP5036, Package_DFN_QFN:VQFN-46-1EP_5x6mm_P0.4mm_EP2.8x3.8mm, F.Cu at (166.0, 88.5)
- added U3: PCM5102AQPWRQ1, Package_SO:TSSOP-20_4.4x6.5mm_P0.65mm, F.Cu at (134.8, 130.5)
- added U4: MCP6004, Package_SO:TSSOP-14_4.4x5mm_P0.65mm, F.Cu at (156.7, 134.5)
- added U5: TL071, Package_SO:SO-8_5.3x6.2mm_P1.27mm, F.Cu at (119.9, 129.5)
- added U6: LM4040DBZ-10, Package_TO_SOT_SMD:SOT-23, F.Cu at (166.6, 127.0)
- added U7: TPS560430, Package_TO_SOT_SMD:SOT-23-6_Handsoldering, F.Cu at (141.2, 100.6)
- added U8: MIC5205-3.3YM5, Package_TO_SOT_SMD:SOT-23-5, F.Cu at (156.6, 127.1)
- added Y1: ABM3-8.000MHZ-D2Y-T, Crystal:Crystal_SMD_5032-2Pin_5.0x3.2mm_HandSoldering, F.Cu at (160.0, 110.2)

Commit message: Routing in progress
Parts:
- removed D33: LED, LED_THT:LED_D3.0mm
- C46: footprint Capacitor_SMD:C_0805_2012Metric_Pad1.18x1.45mm_HandSolder -> Capacitor_Tantalum_SMD:CP_EIA-7343-31_Kemet-D_Pad2.25x2.55mm_HandSolder
- D1, D10, D11, D12, D13, D14, D15, D16, D17, D18, D19, D2, D20, D21, D22, D23, D24, D25, D26, D27, D28, D29, D3, D30, D31, D32, D4, D5, D6, D7, D8, D9: moved to B.Cu
- moved D23 35.1 mm to (159.0, 67.0), turned to 180 degrees
- moved D6 32.1 mm to (152.0, 92.0), turned to 180 degrees
- moved D20 31.1 mm to (134.0, 62.0), turned to 180 degrees
- moved D8 27.8 mm to (141.0, 82.0), turned to 180 degrees
- moved D32 27.7 mm to (134.0, 82.0), turned to 180 degrees
- moved D1 26.7 mm to (159.0, 57.0), turned to 180 degrees
- moved D27 25.1 mm to (152.0, 87.0), turned to 180 degrees
- moved D3 24.8 mm to (159.0, 87.0), turned to 180 degrees
- moved D17 24.5 mm to (141.0, 57.0), turned to 180 degrees
- moved D4 23.4 mm to (152.0, 62.0), turned to 180 degrees
- moved D13 23.0 mm to (159.0, 77.0), turned to 180 degrees
- moved D9 22.5 mm to (134.0, 57.0), turned to 180 degrees
- moved D22 22.1 mm to (134.0, 92.0), turned to 180 degrees
- moved D15 19.7 mm to (152.0, 67.0), turned to 180 degrees
- moved C13 18.4 mm to (177.0, 87.0), turned to 270 degrees
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Connections:
- U2 pad 33: Net-(D33-Pad1) -> (no net)
Routing:
- net GND: track 0.00 -> 517.1 mm, vias 0 -> 34
- net +3.3VA: track 0.00 -> 191.0 mm, vias 0 -> 11
- net /core/ADC_CH7: track 0.00 -> 99.2 mm, vias 0 -> 1
- net +3V3: track 0.00 -> 94.4 mm, vias 0 -> 1
- net /core/ADC_CH8: track 0.00 -> 84.6 mm, vias 0 -> 1
- net /core/ADC_CH6: track 0.00 -> 79.8 mm, vias 0 -> 3
- net AREF_-10: track 0.00 -> 64.7 mm, vias 0 -> 2
- net /core/ADC_CH4: track 0.00 -> 64.5 mm, vias 0 -> 1
- net /core/ADC_CH5: track 0.00 -> 63.1 mm, vias 0 -> 1
- net /core/I2S_SD: track 0.00 -> 61.1 mm, vias 0 -> 2
- net Net-(C40-Pad1): track 0.00 -> 55.0 mm, vias 0 -> 2
- net /core/I2S_WS: track 0.00 -> 54.8 mm, vias 0 -> 2
- net Net-(L3-Pad2): track 0.00 -> 50.4 mm, vias 0 -> 2
- net /core/I2S_CK: track 0.00 -> 48.7 mm, vias 0 -> 2
- net /core/ADC_CH1: track 0.00 -> 45.2 mm, vias 0 -> 4
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Other:
- net class Default: clearance 0.2 -> 0.15; trace_width 0.25 -> 0.15; via_dia 0.8 -> 0.6; via_drill 0.4 -> 0.3
- rule trace_clearance: 0.2 -> 0.15
- rule trace_min: 0.2 -> 0.15
- rule via_min_size: 0.4 -> 0.2

Commit message: Finished routing
Parts:
- C46: footprint Capacitor_Tantalum_SMD:CP_EIA-7343-31_Kemet-D_Pad2.25x2.55mm_HandSolder -> Capacitor_SMD:C_0805_2012Metric_Pad1.18x1.45mm_HandSolder
- moved D22 36.2 mm to (131.8, 55.9), turned to 0 degrees
- moved D9 33.9 mm to (131.8, 90.9), turned to 0 degrees
- moved D11 26.2 mm to (131.8, 60.9), turned to 0 degrees
- moved D20 24.0 mm to (131.8, 85.9), turned to 0 degrees
- moved D32 16.3 mm to (131.8, 65.9), turned to 0 degrees
- moved D31 14.0 mm to (131.8, 80.9), turned to 0 degrees
- moved D21 6.52 mm to (131.8, 70.9), turned to 0 degrees
- moved D10 4.46 mm to (131.8, 75.9), turned to 0 degrees
- moved C8 1.91 mm to (168.7, 103.0)
- moved SW3 1.54 mm to (144.9, 48.5)
- moved C9 1.37 mm to (168.7, 105.0)
- moved D1 1.12 mm to (158.9, 55.9)
- moved D12 1.12 mm to (158.9, 60.9)
- moved D17 1.12 mm to (140.9, 55.9)
- moved D25 1.12 mm to (151.9, 55.9)
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Connections:
- U1 pad 2: (no net) -> Net-(SW3-Pad2)
- U1 pad 20: Net-(SW3-Pad2) -> (no net)
Routing:
- net +3V3: track 94.4 -> 364.3 mm, vias 1 -> 4
- net GND: track 517.1 -> 675.6 mm, vias 34 -> 64
- net Net-(SW2-Pad2): track 7.20 -> 106.6 mm, vias 0 -> 1
- net Net-(D11-Pad1): track 0.00 -> 76.5 mm
- net Net-(SW3-Pad2): track 7.20 -> 82.0 mm, vias 0 -> 1
- net Net-(SW1-Pad2): track 0.00 -> 74.5 mm, vias 0 -> 1
- net Net-(D32-Pad1): track 0.00 -> 70.3 mm
- net +3.3VA: track 191.0 -> 260.2 mm
- net Net-(D21-Pad1): track 0.00 -> 64.1 mm
- net Net-(D22-Pad1): track 0.00 -> 62.0 mm, vias 0 -> 1
- net Net-(D10-Pad1): track 0.00 -> 57.8 mm
- net Net-(D31-Pad1): track 0.00 -> 51.6 mm
- net Net-(D17-Pad1): track 0.00 -> 48.6 mm
- net Net-(D20-Pad1): track 0.00 -> 45.3 mm
- net /core/LEDS_SDA: track 0.00 -> 43.9 mm
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- added copper zone on B.Cu, net GND
- added copper zone on F.Cu, net GND
Other:
- board text added: "URSAE"
- board text added: "rev. 0.0.1"

Commit message: Alpha v0.0.1
Parts:
- moved R14 1.93 mm to (145.5, 136.7), turned to 180 degrees
Routing:
- net AREF_-10: track 64.7 -> 62.0 mm
- net Net-(C30-Pad2): track 16.7 -> 17.5 mm
- net GND: track 675.6 -> 674.9 mm, vias 64 -> 87
- net Net-(D22-Pad1): track 62.0 -> 62.5 mm
